File: pcb/tyre_temp_sense/tyre_temp_sense.sch (KiCad schematic (older format))
At the start: 40 parts, among them J1 POWER & CAN, J2 Extra i2c ports (no pullups), J3 Analog breakout, J4 MUX Port 0, J5 MUX Port 1, J6 MUX Port 2, J7 MUX Port 3, J8 Conn_01x02, U1 TCA9548APWR, U2 MCP2515-I/ST, U3 MCP2551-I-SN, Y1 8 mhz

Commit message: PCB design complete
Parts:
- removed C2: 30pF, Capacitor_SMD:C_0603_1608Metric, symbol Device:C
- removed J2: Extra i2c ports (no pullups), Connector_PinHeader_2.54mm:PinHeader_1x08_P2.54mm_Vertical, symbol Connector:Conn_01x08_Male
- added C2: 30p, Capacitor_SMD:C_0603_1608Metric, symbol tyre_temp_sense-rescue:C-Device
- added J2: 5V, Connector_PinHeader_2.54mm:PinHeader_1x04_P2.54mm_Vertical, symbol tyre_temp_sense-rescue:Conn_01x04_Male-Connector
- added J9: GND, Connector_PinHeader_2.54mm:PinHeader_1x04_P2.54mm_Vertical, symbol tyre_temp_sense-rescue:Conn_01x04_Male-Connector
- A1: symbol MCU_Module:Arduino_Nano_v3.x -> tyre_temp_sense-rescue:Arduino_Nano_v3.x-MCU_Module
- C1, C4: symbol Device:C -> tyre_temp_sense-rescue:C-Device
- C3: value 30pF -> 30p; symbol Device:C -> tyre_temp_sense-rescue:C-Device
- J1, J4, J5, J6, J7: symbol Connector_Generic:Conn_01x04 -> tyre_temp_sense-rescue:Conn_01x04-Connector_Generic
- J3: value Analog breakout -> Analog; symbol Connector:Conn_01x04_Male -> tyre_temp_sense-rescue:Conn_01x04_Male-Connector
- J8: symbol Connector_Generic:Conn_01x02 -> tyre_temp_sense-rescue:Conn_01x02-Connector_Generic
- R1, R10, R11, R12, R13, R14, R2, R3, R4, R5, R6, R7, R8, R9: symbol Device:R -> tyre_temp_sense-rescue:R-Device
- TP1: value CAN_H -> CAN+; symbol Connector:TestPoint -> tyre_temp_sense-rescue:TestPoint-Connector
- TP2, TP4, TP5, TP6, TP7, TP8, TP9: symbol Connector:TestPoint -> tyre_temp_sense-rescue:TestPoint-Connector
- TP3: value CAN_L -> CAN-; symbol Connector:TestPoint -> tyre_temp_sense-rescue:TestPoint-Connector
- U1: symbol Interface_Expansion:TCA9548APWR -> tyre_temp_sense-rescue:TCA9548APWR-Interface_Expansion
- U2: symbol Interface_CAN_LIN:MCP2515-xST -> tyre_temp_sense-rescue:MCP2515-xST-Interface_CAN_LIN
- U3: symbol Interface_CAN_LIN:MCP2551-I-SN -> tyre_temp_sense-rescue:MCP2551-I-SN-Interface_CAN_LIN
- Y1: footprint (none) -> Crystal:Crystal_SMD_5032-2Pin_5.0x3.2mm; symbol Device:Crystal -> tyre_temp_sense-rescue:Crystal-Device; JLCPCB Part # C403948 -> C115962
Connections:
- net +3V3: now also J4.3 (Pin_3), J5.3 (Pin_3), J6.3 (Pin_3), J7.3 (Pin_3); no longer J4.2 (Pin_2), J5.2 (Pin_2), J6.2 (Pin_2), J7.2 (Pin_2)
- net +5V: now also J2.1 (Pin_1), J2.2 (Pin_2), J2.3 (Pin_3), J2.4 (Pin_4)
- net GND: now also J4.4 (Pin_4), J5.4 (Pin_4), J6.4 (Pin_4), J7.4 (Pin_4), C2.2, J9.1 (Pin_1), J9.2 (Pin_2), J9.3 (Pin_3), J9.4 (Pin_4); no longer J4.1 (Pin_1), J5.1 (Pin_1), J6.1 (Pin_1), J7.1 (Pin_1)
- net A0: now reaches A1.19 (A0), J3.4 (Pin_4)
- net A1: now reaches A1.20 (A1), J3.3 (Pin_3)
- net A2: now reaches A1.21 (A2), J3.2 (Pin_2)
- net A3: now reaches A1.22 (A3), J3.1 (Pin_1)
- net at U2.8 (OSC2): now also Y1.2, C2.1; no longer Y1.1
- net at C3.1, U2.9 (OSC1): now also Y1.1; no longer Y1.2
- net at R11.2, U1.10 (SD3): now also J7.1 (Pin_1); no longer J7.4 (Pin_4)
- net at R10.2, U1.11 (SC3): now also J7.2 (Pin_2); no longer J7.3 (Pin_3)
- net at R5.2, U1.4 (SD0): now also J4.1 (Pin_1); no longer J4.4 (Pin_4)
- net at R4.2, U1.5 (SC0): now also J4.2 (Pin_2); no longer J4.3 (Pin_3)
- net at R7.2, U1.6 (SD1): now also J5.1 (Pin_1); no longer J5.4 (Pin_4)
- net at R6.2, U1.7 (SC1): now also J5.2 (Pin_2); no longer J5.3 (Pin_3)
- net at R9.2, U1.8 (SD2): now also J6.1 (Pin_1); no longer J6.4 (Pin_4)
- net at R8.2, U1.9 (SC2): now also J6.2 (Pin_2); no longer J6.3 (Pin_3)
- net CAN_H renamed CAN+
- net CAN+: now also J1.3 (Pin_3), TP3.1; no longer J1.4 (Pin_4), TP1.1
- net CAN_L renamed CAN-
- net CAN-: now also J1.4 (Pin_4), TP1.1; no longer J1.3 (Pin_3), TP3.1
- no-connect marks 20 -> 28
Other:
- note added: "Breakouts"
- note removed: "Breakout extra i2c connections\n"
- moved on the sheet: C1, C3, J3, J4, J5, J6, J7, R1, R10, R11, R2, R3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
