File: pcb/tyre_temp_sense/tyre_temp_sense.kicad_pcb (KiCad board)
At the start: 2 copper layers, 184 x 60.5 mm, 19 parts, among them J2 POWER & CAN, J8 Conn_01x02, U1 TCA9548APWR, U2 MCP2515-xST, U3 MCP2551-I-SN

Commit message: Updates
Parts:
- added C1: 10uF, Capacitor_SMD:C_0603_1608Metric, F.Cu at (224.0, 99.5)
- added C2: 30pF, Capacitor_SMD:C_0603_1608Metric, F.Cu at (221.5, 43.0)
- added C3: 30pF, Capacitor_SMD:C_0603_1608Metric, F.Cu at (216.5, 43.0)
- added C4: 0.1uF, Capacitor_SMD:C_0603_1608Metric, F.Cu at (224.0, 60.0)
- added J1: POWER & CAN, Connector_JST:JST_EH_B4B-EH-A_1x04_P2.50mm_Vertical, F.Cu at (234.5, 60.5)
- added J3: Analog breakout, Connector_JST:JST_EH_B4B-EH-A_1x04_P2.50mm_Vertical, F.Cu at (193.0, 53.0)
- added J4: MUX Port 0, Connector_JST:JST_EH_B4B-EH-A_1x04_P2.50mm_Vertical, F.Cu at (234.5, 92.5)
- added J5: MUX Port 1, Connector_JST:JST_EH_B4B-EH-A_1x04_P2.50mm_Vertical, F.Cu at (234.5, 85.5)
- added J6: MUX Port 2, Connector_JST:JST_EH_B4B-EH-A_1x04_P2.50mm_Vertical, F.Cu at (234.5, 78.0)
- added J7: MUX Port 3, Connector_JST:JST_EH_B4B-EH-A_1x04_P2.50mm_Vertical, F.Cu at (234.5, 70.5)
- added R1: 10K, Resistor_SMD:R_0603_1608Metric, F.Cu at (208.2, 116.0)
- added R10: 4.7K, Resistor_SMD:R_0603_1608Metric, F.Cu at (222.0, 111.9)
- added R11: 4.7K, Resistor_SMD:R_0603_1608Metric, F.Cu at (230.7, 117.0)
- added R12: 10K, Resistor_SMD:R_0603_1608Metric, F.Cu at (105.0, 82.0)
- added R13: 10K, Resistor_SMD:R_0603_1608Metric, F.Cu at (235.2, 27.0)
- added R14: 120, Resistor_SMD:R_0603_1608Metric, F.Cu at (225.0, 34.0)
- added R2: 4.7K, Resistor_SMD:R_0603_1608Metric, F.Cu at (232.0, 112.5)
- added R3: 4.7K, Resistor_SMD:R_0603_1608Metric, F.Cu at (218.0, 111.9)
- added R4: 4.7K, Resistor_SMD:R_0603_1608Metric, F.Cu at (225.7, 118.5)
- added R5: 4.7K, Resistor_SMD:R_0603_1608Metric, F.Cu at (221.2, 116.5)
- added R6: 4.7K, Resistor_SMD:R_0603_1608Metric, F.Cu at (215.5, 115.5)
- added R7: 4.7K, Resistor_SMD:R_0603_1608Metric, F.Cu at (214.0, 111.9)
- added R8: 4.7K, Resistor_SMD:R_0603_1608Metric, F.Cu at (235.2, 116.0)
- added R9: 4.7K, Resistor_SMD:R_0603_1608Metric, F.Cu at (226.2, 114.0)
- added Y1: 8 mhz, Crystal:Crystal_SMD_3225-4Pin_3.2x2.5mm, F.Cu at (215.1, 52.9)
- J2: value POWER & CAN -> Extra i2c ports (no pullups); footprint Connector_JST:JST_EH_B4B-EH-A_1x04_P2.50mm_Vertical -> Connector_JST:JST_EH_B8B-EH-A_1x08_P2.50mm_Vertical
- TP1: value TestPoint -> CAN_H
- TP2: value TestPoint -> GND
- TP3: value TestPoint -> CAN_L
- TP4: value TestPoint -> 5V
- TP5: value TestPoint -> MOSI
- TP6: value TestPoint -> MISO
- TP7: value TestPoint -> CLK
- TP8: value TestPoint -> RX
- TP9: value TestPoint -> TX
- U2: value MCP2515-xST -> MCP2515-I/ST
- moved U3 115.5 mm to (234.5, 52.0)
- moved TP1 114.3 mm to (237.0, 38.0)
- moved J2 100.8 mm to (210.0, 92.5)
- moved U1 97.4 mm to (226.0, 84.0), turned to 180 degrees
- moved J8 93.2 mm to (216.0, 32.0)
- moved A1 83.9 mm to (176.0, 82.5), turned to 90 degrees
- moved U2 80.8 mm to (223.5, 52.0)
- moved TP6 36.4 mm to (101.5, 94.5)
- moved TP9 33.3 mm to (143.9, 52.7)
- moved TP7 27.3 mm to (119.5, 92.0)
- moved TP2 13.5 mm to (115.5, 60.5)
- moved TP5 11.6 mm to (113.2, 77.8)
- moved TP4 9.64 mm to (129.2, 61.0)
- moved TP3 9.41 mm to (117.3, 75.3)
- moved TP8 4.16 mm to (119.9, 70.2)
Connections:
- J2 pad 1: GND -> Net-(J2-Pad1)
- J2 pad 2: +5V -> Net-(J2-Pad2)
- J2 pad 3: CAN_L -> Net-(J2-Pad3)
- J2 pad 4: CAN_H -> Net-(J2-Pad4)
- TP1 pad 1: MOSI_CAN -> CAN_H
- TP2 pad 1: MISO_CAN -> GND
- TP3 pad 1: CLK_CAN -> CAN_L
- TP4 pad 1: Net-(A1-Pad2) -> +5V
- TP5 pad 1: Net-(A1-Pad1) -> MOSI_CAN
- TP6 pad 1: CAN_H -> MISO_CAN
- TP7 pad 1: GND -> CLK_CAN
- TP8 pad 1: CAN_L -> Net-(A1-Pad2)
- TP9 pad 1: +5V -> Net-(A1-Pad1)
- U1 pad 13: Net-(J3-Pad7) -> Net-(J2-Pad1)
- U1 pad 14: Net-(J3-Pad8) -> Net-(J2-Pad2)
- U1 pad 15: Net-(J3-Pad5) -> Net-(J2-Pad3)
- U1 pad 16: Net-(J3-Pad6) -> Net-(J2-Pad4)
- U1 pad 17: Net-(J3-Pad3) -> Net-(J2-Pad5)
- U1 pad 18: Net-(J3-Pad4) -> Net-(J2-Pad6)
- U1 pad 19: Net-(J3-Pad1) -> Net-(J2-Pad7)
- U1 pad 20: Net-(J3-Pad2) -> Net-(J2-Pad8)
Other:
- outline, holes or cut-outs redrawn

Commit message: PCB design complete
Parts:
- removed the REF** at (69.0, 102.0)
- removed the REF** at (245.0, 102.0)
- removed the REF** at (245.0, 49.5)
- removed the REF** at (69.0, 49.5)
- added ?: , , F.Cu at (79.5, 101.6)
- added ?: , , F.Cu at (80.3, 101.9)
- added J9: GND, Connector_PinHeader_2.54mm:PinHeader_1x04_P2.54mm_Vertical, F.Cu at (97.2, 94.0)
- added REF**: MountingHole_3.2mm_M3, MountingHole:MountingHole_3.2mm_M3, F.Cu at (116.0, 101.0)
- added REF**: MountingHole_3.2mm_M3, MountingHole:MountingHole_3.2mm_M3, F.Cu at (116.0, 44.0)
- added REF**: MountingHole_3.2mm_M3, MountingHole:MountingHole_3.2mm_M3, F.Cu at (74.0, 44.0)
- added REF**: MountingHole_3.2mm_M3, MountingHole:MountingHole_3.2mm_M3, F.Cu at (74.0, 101.0)
- C2, C3: value 30pF -> 30p
- J2: value Extra i2c ports (no pullups) -> 5V; footprint Connector_JST:JST_EH_B8B-EH-A_1x08_P2.50mm_Vertical -> Connector_PinHeader_2.54mm:PinHeader_1x04_P2.54mm_Vertical
- J3: value Analog breakout -> Analog; footprint Connector_JST:JST_EH_B4B-EH-A_1x04_P2.50mm_Vertical -> Connector_PinHeader_2.54mm:PinHeader_1x04_P2.54mm_Vertical
- TP1: value CAN_H -> CAN+
- TP3: value CAN_L -> CAN-
- Y1: footprint Crystal:Crystal_SMD_3225-4Pin_3.2x2.5mm -> Crystal:Crystal_SMD_5032-2Pin_5.0x3.2mm
- moved R2 140.3 mm to (96.6, 75.5), turned to 90 degrees
- moved U3 138.6 mm to (96.0, 55.9)
- moved R13 136.5 mm to (101.1, 52.8), turned to 90 degrees
- moved C1 133.3 mm to (92.8, 75.5), turned to 90 degrees
- moved C2 132.9 mm to (88.6, 42.4), turned to 90 degrees
- moved C3 131.7 mm to (84.8, 42.4), turned to 90 degrees
- moved R11 131.5 mm to (108.4, 68.6), turned to 180 degrees
- moved U1 130.8 mm to (96.0, 69.2)
- moved R8 129.1 mm to (111.8, 78.2)
- moved Y1 128.6 mm to (86.7, 45.8)
- moved R3 128.5 mm to (94.7, 75.5), turned to 90 degrees
- moved J1 128.2 mm to (106.7, 50.8)
- moved C4 128.2 mm to (97.0, 42.5), turned to 90 degrees
- moved J7 128.0 mm to (106.7, 63.5)
- moved J6 127.9 mm to (106.7, 73.2)
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Connections:
- net Net-(A1-Pad19) renamed A0
- net Net-(A1-Pad20) renamed A1
- net Net-(A1-Pad21) renamed A2
- net Net-(A1-Pad22) renamed A3
- J1 pad 3: CAN_L -> CAN+
- J1 pad 4: CAN_H -> CAN-
- J2 pad 1: Net-(J2-Pad1) -> +5V
- J2 pad 2: Net-(J2-Pad2) -> +5V
- J2 pad 3: Net-(J2-Pad3) -> +5V
- J2 pad 4: Net-(J2-Pad4) -> +5V
- J4 pad 1: GND -> Net-(J4-Pad1)
- J4 pad 2: +3V3 -> Net-(J4-Pad2)
- J4 pad 3: Net-(J4-Pad3) -> +3V3
- J4 pad 4: Net-(J4-Pad4) -> GND
- J5 pad 1: GND -> Net-(J5-Pad1)
- J5 pad 2: +3V3 -> Net-(J5-Pad2)
- J5 pad 3: Net-(J5-Pad3) -> +3V3
- J5 pad 4: Net-(J5-Pad4) -> GND
- J6 pad 1: GND -> Net-(J6-Pad1)
- J6 pad 2: +3V3 -> Net-(J6-Pad2)
- J6 pad 3: Net-(J6-Pad3) -> +3V3
- J6 pad 4: Net-(J6-Pad4) -> GND
- J7 pad 1: GND -> Net-(J7-Pad1)
- J7 pad 2: +3V3 -> Net-(J7-Pad2)
- J7 pad 3: Net-(J7-Pad3) -> +3V3
- J7 pad 4: Net-(J7-Pad4) -> GND
- J8 pad 2: CAN_L -> CAN-
- R10 pad 2: Net-(J7-Pad3) -> Net-(J7-Pad2)
- R11 pad 2: Net-(J7-Pad4) -> Net-(J7-Pad1)
- R14 pad 2: CAN_H -> CAN+
- R4 pad 2: Net-(J4-Pad3) -> Net-(J4-Pad2)
- R5 pad 2: Net-(J4-Pad4) -> Net-(J4-Pad1)
- R6 pad 2: Net-(J5-Pad3) -> Net-(J5-Pad2)
- R7 pad 2: Net-(J5-Pad4) -> Net-(J5-Pad1)
- R8 pad 2: Net-(J6-Pad3) -> Net-(J6-Pad2)
- R9 pad 2: Net-(J6-Pad4) -> Net-(J6-Pad1)
- TP1 pad 1: CAN_H -> CAN-
- TP3 pad 1: CAN_L -> CAN+
- U1 pad 10: Net-(J7-Pad4) -> Net-(J7-Pad1)
- U1 pad 11: Net-(J7-Pad3) -> Net-(J7-Pad2)
- U1 pad 13: Net-(J2-Pad1) -> Net-(U1-Pad13)
- U1 pad 14: Net-(J2-Pad2) -> Net-(U1-Pad14)
- U1 pad 15: Net-(J2-Pad3) -> Net-(U1-Pad15)
- U1 pad 16: Net-(J2-Pad4) -> Net-(U1-Pad16)
- U1 pad 17: Net-(J2-Pad5) -> Net-(U1-Pad17)
- U1 pad 18: Net-(J2-Pad6) -> Net-(U1-Pad18)
- U1 pad 19: Net-(J2-Pad7) -> Net-(U1-Pad19)
- U1 pad 20: Net-(J2-Pad8) -> Net-(U1-Pad20)
- U1 pad 4: Net-(J4-Pad4) -> Net-(J4-Pad1)
- U1 pad 5: Net-(J4-Pad3) -> Net-(J4-Pad2)
- U1 pad 6: Net-(J5-Pad4) -> Net-(J5-Pad1)
- U1 pad 7: Net-(J5-Pad3) -> Net-(J5-Pad2)
- U1 pad 8: Net-(J6-Pad4) -> Net-(J6-Pad1)
- U1 pad 9: Net-(J6-Pad3) -> Net-(J6-Pad2)
- U3 pad 6: CAN_L -> CAN-
- U3 pad 7: CAN_H -> CAN+
- Y1 pad 1: Net-(C2-Pad1) -> Net-(C3-Pad1)
- Y1 pad 2: Net-(C3-Pad1) -> Net-(C2-Pad1)
Routing:
- net +5V: track 0.00 -> 246.6 mm, vias 0 -> 5
- net MOSI_CAN: track 0.00 -> 80.4 mm, vias 0 -> 1
- net MISO_CAN: track 0.00 -> 69.6 mm, vias 0 -> 1
- net CLK_CAN: track 0.00 -> 63.8 mm, vias 0 -> 1
- net +3V3: track 0.00 -> 52.6 mm
- net D6: track 0.00 -> 50.2 mm, vias 0 -> 1
- net D2: track 0.00 -> 45.7 mm, vias 0 -> 1
- net CAN-: track 0.00 -> 36.2 mm, vias 0 -> 1
- net Net-(J4-Pad2): track 0.00 -> 33.7 mm
- net CAN+: track 0.00 -> 32.7 mm, vias 0 -> 2
- net Net-(J4-Pad1): track 0.00 -> 30.7 mm
- net GND: track 0.00 -> 27.6 mm, vias 0 -> 29
- net Net-(J5-Pad2): track 0.00 -> 25.2 mm
- net Net-(J5-Pad1): track 0.00 -> 22.5 mm
- net A0: track 0.00 -> 21.4 mm
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- added copper zone on B.Cu, net GND
Other:
- board size 184 x 60.5 mm -> 50 x 65 mm
- board text added: "120Ω"
- board text added: "5V"
- board text added: "A0"
- board text added: "A1"
- board text added: "A2"
- board text added: "A3"
- board text added: "AUMT 2021 Tyre Temp Bryce Chung"
- board text added: "Arduino is wet Arduino is dry Arduino is warm"
- board text added: "CANH"
- board text added: "CAN_L"
- board text added: "CLK"
- board text added: "DATA CLK 3V3 GND"
- board text added: "Debug Table Condition Issue"
- board text added: "GND"
- board text added: "MISO"
- board text added: "MOSI"
- board text added: "RX"
- board text added: "Raining Not raining Australia"
- board text added: "TX"

Commit message: First revision, ready for production
Added JLCPCB parts

rev 1

Revert "rev 1"

This reverts commit d7fe8d90d780ed24d08af68c791964fcba5617af.

Revert "Revert "rev 1""

This reverts commit 5d4b21aec522fc29a8afe0da54f0448a4a3d7d19.
Parts:
- C2, C3: value 30p -> 30pF
- C4: value 0.1uF -> 10uF
- R1, R12: value 10K -> 10k
- R10, R11, R2, R3, R4, R5, R6, R7, R8, R9: value 4.7K -> 4.7k
Routing:
- net MOSI_CAN: track 80.4 -> 76.1 mm
Other:
- board text added: "CANL"
- board text added: "JLCJLCJLCJLC"
- board text removed: "CAN_L"
