File: pcb/tyre_temp_sense/tyre_temp_sense(with mounts).kicad_pcb (KiCad board)
At the start: 2 copper layers, 50 x 65 mm, 47 parts, among them J1 POWER & CAN, J2 5V, J3 Analog, J4 MUX Port 0, J5 MUX Port 1, J6 MUX Port 2, J7 MUX Port 3, J8 Conn_01x02, J9 GND, U1 TCA9548APWR, U2 MCP2515-I/ST, U3 MCP2551-I-SN, Y1 8 mhz

Commit message: Revert "rev 1"
This reverts commit d7fe8d90d780ed24d08af68c791964fcba5617af.
Parts:
- added J1: Molex, Connector_Molex:Molex_Micro-Fit_3.0_43650-0415_1x04_P3.00mm_Vertical, B.Cu at (125.5, 60.2)
- added J1: Molex, Connector_Molex:Molex_Micro-Fit_3.0_43650-0415_1x04_P3.00mm_Vertical, B.Cu at (125.5, 86.9)
- added J2: MLX Sensor, Package_TO_SOT_THT:TO-39-4_Window, F.Cu at (132.1, 64.8)
- added J2: MLX Sensor, Package_TO_SOT_THT:TO-39-4_Window, F.Cu at (132.1, 91.4)
- added REF**: MountingHole_3.2mm_M3, MountingHole:MountingHole_3.2mm_M3, F.Cu at (134.0, 54.8)
- added REF**: MountingHole_3.2mm_M3, MountingHole:MountingHole_3.2mm_M3, F.Cu at (134.0, 74.3)
- added REF**: MountingHole_3.2mm_M3, MountingHole:MountingHole_3.2mm_M3, F.Cu at (134.0, 81.5)
- added REF**: MountingHole_3.2mm_M3, MountingHole:MountingHole_3.2mm_M3, F.Cu at (134.0, 101.0)
Routing:
- net (no net): track 0.00 -> 99.9 mm
Other:
- board size 50 x 65 mm -> 71.8 x 65 mm
